File: KiCad/Sequencer/Sequencer.kicad_sch (KiCad schematic)
At the start: 50 parts, among them J1 Eurorack Power, J2 AudioJack, SW1 SW_Push, U1 TL072, U2 4017, U3 TL074, U4 TL074, U5 TL072, U6 TL072

Commit message: V1.0 Schematic Finished
Parts:
- removed R27: 40k, symbol Device:R
- added RV12: 5k, symbol Device:R_Potentiometer_Trim
- added RV13: 10k, symbol Device:R_Potentiometer_Trim
- C1: value 10u -> 1u
- R1: value 1k -> 39k
- RV1: value 100k -> 1M
Connections:
- net at R26.2, U6.2 (-): now also RV13.2
- net at RV1.1: now also RV12.2; no longer R1.2
- net at U6.1, U6.5 (+): now also R1.1
- net at C1.1, U1.2 (-): now also RV12.1; no longer R1.1
- new net: R1.2, RV13.3
- no-connect marks 2 -> 4
Other:
- note added: "Trim Poti to set highest freq to 200Hz"
- note added: "Trim Poti to set the output voltage to max +5V"
- title: Basic Sequencer -> CD4017 10-Step Sequencer

Commit message: Finished Version 1.0 of PCB
Parts:
- removed J1: Eurorack Power, symbol Connector_Generic:Conn_02x05_Counter_Clockwise
- added J1: Eurorack Power, Connector_PinHeader_2.54mm:PinHeader_2x05_P2.54mm_Vertical, symbol Connector_Generic:Conn_02x05_Odd_Even
- C1: footprint (none) -> Capacitor_SMD:C_0805_2012Metric_Pad1.18x1.45mm_HandSolder
- D1, D10, D11, D2, D3, D4, D5, D6, D7, D8, D9: footprint (none) -> Diode_THT:D_DO-34_SOD68_P2.54mm_Vertical_AnodeUp
- J2: footprint (none) -> Connector_Audio:Jack_3.5mm_QingPu_WQP-PJ398SM_Vertical_CircularHoles
- R1: renamed from R3; footprint (none) -> Resistor_SMD:R_0805_2012Metric_Pad1.20x1.40mm_HandSolder
- R15: renamed from R6; footprint (none) -> Resistor_SMD:R_0805_2012Metric_Pad1.20x1.40mm_HandSolder
- R16: renamed from R7; footprint (none) -> Resistor_SMD:R_0805_2012Metric_Pad1.20x1.40mm_HandSolder
- R17: renamed from R8; footprint (none) -> Resistor_SMD:R_0805_2012Metric_Pad1.20x1.40mm_HandSolder
- R18: renamed from R9; footprint (none) -> Resistor_SMD:R_0805_2012Metric_Pad1.20x1.40mm_HandSolder
- R19: renamed from R10; footprint (none) -> Resistor_SMD:R_0805_2012Metric_Pad1.20x1.40mm_HandSolder
- R2: renamed from R4; footprint (none) -> Resistor_SMD:R_0805_2012Metric_Pad1.20x1.40mm_HandSolder
- R20: renamed from R11; footprint (none) -> Resistor_SMD:R_0805_2012Metric_Pad1.20x1.40mm_HandSolder
- R21: renamed from R12; footprint (none) -> Resistor_SMD:R_0805_2012Metric_Pad1.20x1.40mm_HandSolder
- R22: renamed from R13; footprint (none) -> Resistor_SMD:R_0805_2012Metric_Pad1.20x1.40mm_HandSolder
- R23: renamed from R14; footprint (none) -> Resistor_SMD:R_0805_2012Metric_Pad1.20x1.40mm_HandSolder
- R24: renamed from R15; footprint (none) -> Resistor_SMD:R_0805_2012Metric_Pad1.20x1.40mm_HandSolder
- R25: renamed from R16; footprint (none) -> Resistor_SMD:R_0805_2012Metric_Pad1.20x1.40mm_HandSolder
- R26: renamed from R17; footprint (none) -> Resistor_SMD:R_0805_2012Metric_Pad1.20x1.40mm_HandSolder
- R27: renamed from R18; footprint (none) -> Resistor_SMD:R_0805_2012Metric_Pad1.20x1.40mm_HandSolder
- R28: renamed from R19; footprint (none) -> Resistor_SMD:R_0805_2012Metric_Pad1.20x1.40mm_HandSolder
- R29: renamed from R20; footprint (none) -> Resistor_SMD:R_0805_2012Metric_Pad1.20x1.40mm_HandSolder
- R3: renamed from R5; footprint (none) -> Resistor_SMD:R_0805_2012Metric_Pad1.20x1.40mm_HandSolder
- R30: renamed from R21; footprint (none) -> Resistor_SMD:R_0805_2012Metric_Pad1.20x1.40mm_HandSolder
- R31: renamed from R22; footprint (none) -> Resistor_SMD:R_0805_2012Metric_Pad1.20x1.40mm_HandSolder
- R32: renamed from R23; footprint (none) -> Resistor_SMD:R_0805_2012Metric_Pad1.20x1.40mm_HandSolder
- R33: renamed from R24; footprint (none) -> Resistor_SMD:R_0805_2012Metric_Pad1.20x1.40mm_HandSolder
- R34: renamed from R25; footprint (none) -> Resistor_SMD:R_0805_2012Metric_Pad1.20x1.40mm_HandSolder
- R35: renamed from R26; footprint (none) -> Resistor_SMD:R_0805_2012Metric_Pad1.20x1.40mm_HandSolder
- R36: renamed from R1; value 39k -> 33k; footprint (none) -> Resistor_SMD:R_0805_2012Metric_Pad1.20x1.40mm_HandSolder
- R37: renamed from R28; footprint (none) -> Resistor_SMD:R_0805_2012Metric_Pad1.20x1.40mm_HandSolder
- R4: renamed from R2; footprint (none) -> Resistor_SMD:R_0805_2012Metric_Pad1.20x1.40mm_HandSolder
- RV1: renamed from RV12; footprint (none) -> Potentiometer_THT:Potentiometer_Piher_PT-6-V_Vertical
- RV13: value 10k -> 20k; footprint (none) -> Potentiometer_THT:Potentiometer_Piher_PT-6-V_Vertical
- RV2: renamed from RV1; footprint (none) -> Project_Footprints:Potis
- SW1: footprint (none) -> Button_Switch_THT:SW_PUSH_1P1T_6x3.5mm_H4.3_APEM_MJTP1243
- U1, U5, U6: footprint (none) -> Package_DIP:DIP-8_W7.62mm
- U2: footprint (none) -> Package_DIP:DIP-16_W7.62mm
- U3, U4: footprint (none) -> Package_DIP:DIP-14_W7.62mm
Connections:
- net +12V: now also J1.1 (Pin_1), J1.2 (Pin_2)
- net -12V: now also J1.10 (Pin_10), J1.9 (Pin_9)
- net GND: now also J1.3 (Pin_3), J1.4 (Pin_4), J1.5 (Pin_5), J1.6 (Pin_6), J1.7 (Pin_7), J1.8 (Pin_8)
