File: KiCad/Sequencer/Volume_Stage.kicad_sch (KiCad schematic)
At the start: 20 parts

Commit message: V1.0 Schematic Finished
Other:
- company: (none) -> Christian Hickstein
- title: (none) -> CD4017 10-Step Sequencer
Changed lines of the file:
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@@
 	(generator_version "9.0")
 	(paper "A5")
+	(title_block
+		(title "CD4017 10-Step Sequencer")
+		(date "2026-03-06")
+		(rev "1.0")
+		(company "Christian Hickstein")
+		(comment 1 "Volume Stage")
+	)
 	(junction
 		(at 57.15 53.34)

Commit message: Finished Version 1.0 of PCB
Parts:
- R10: renamed from R48; footprint (none) -> Resistor_SMD:R_0805_2012Metric_Pad1.20x1.40mm_HandSolder
- R11: renamed from R49; footprint (none) -> Resistor_SMD:R_0805_2012Metric_Pad1.20x1.40mm_HandSolder
- R12: renamed from R56; footprint (none) -> Resistor_SMD:R_0805_2012Metric_Pad1.20x1.40mm_HandSolder
- R13: renamed from R57; footprint (none) -> Resistor_SMD:R_0805_2012Metric_Pad1.20x1.40mm_HandSolder
- R14: renamed from R58; footprint (none) -> Resistor_SMD:R_0805_2012Metric_Pad1.20x1.40mm_HandSolder
- R5: renamed from R35; footprint (none) -> Resistor_SMD:R_0805_2012Metric_Pad1.20x1.40mm_HandSolder
- R6: renamed from R36; footprint (none) -> Resistor_SMD:R_0805_2012Metric_Pad1.20x1.40mm_HandSolder
- R7: renamed from R37; footprint (none) -> Resistor_SMD:R_0805_2012Metric_Pad1.20x1.40mm_HandSolder
- R8: renamed from R46; footprint (none) -> Resistor_SMD:R_0805_2012Metric_Pad1.20x1.40mm_HandSolder
- R9: renamed from R47; footprint (none) -> Resistor_SMD:R_0805_2012Metric_Pad1.20x1.40mm_HandSolder
- RV10: renamed from RV9; footprint (none) -> Project_Footprints:Potis
- RV11: renamed from RV10; footprint (none) -> Project_Footprints:Potis
- RV12: renamed from RV11; footprint (none) -> Project_Footprints:Potis
- RV3: renamed from RV2; footprint (none) -> Project_Footprints:Potis
- RV4: renamed from RV3; footprint (none) -> Project_Footprints:Potis
- RV5: renamed from RV4; footprint (none) -> Project_Footprints:Potis
- RV6: renamed from RV5; footprint (none) -> Project_Footprints:Potis
- RV7: renamed from RV6; footprint (none) -> Project_Footprints:Potis
- RV8: renamed from RV7; footprint (none) -> Project_Footprints:Potis
- RV9: renamed from RV8; footprint (none) -> Project_Footprints:Potis
